Commit message: m5 urdf

File: Milestone5/wx250s_viz/urdf/wx250s.urdf.xacro (robot description, xacro)
@@ -123,5 +123,5 @@
     <child link="link2" />
     <origin xyz="0 0 ${L1_HEIGHT}" rpy="0 0 0" />
-    <axis xyz="0 1 0" />
+    <axis xyz="0 ${-1} 0" />
     <limit lower="${J2_MIN}" upper="${J2_MAX}" effort="1" velocity="1" />
   </joint>
@@ -130,5 +130,5 @@
     <child link="link3" />
     <origin xyz="0 0 ${L2_HEIGHT}" rpy="0 0 0" />
-    <axis xyz="0 1 0" />
+    <axis xyz="0 ${-1} 0" />
     <limit lower="${J3_MIN}" upper="${J3_MAX}" effort="1" velocity="1" />
   </joint>
@@ -144,5 +144,5 @@
     <child link="link5" />
     <origin xyz="${L4_HEIGHT} 0 0" rpy="0 0 0" />
-    <axis xyz="0 1 0" />
+    <axis xyz="0 ${-1} 0" />
     <limit lower="${J5_MIN}" upper="${J5_MAX}" effort="1" velocity="1" />
   </joint>
